File: PSU200A_Ctrl.brd (EAGLE design)
At the start: 100 x 80 mm, 30 parts, among them IC1 LM358D, IC2 LM358D, U1 LM4040

Commit message: schematic done
Parts:
- added C10, C11, C12, C13, C7: 0.1u, rcl:C1206
- added C8, C9: 1n, rcl:C1206
- added D1: 1N4148DO35-7, diode:DO35-7
- added U2: LM4040, PSU200A_Ctrl:TO92-
- C1: value 2.2u -> 0.1u
- C2: value 1n -> 0.1u
- C3: value 1n -> 2.2u
- C4, C5: value (none) -> 22u; device rcl:C1206 -> rcl:PANASONIC_B
- C6: value (none) -> 0.1u
- R4: value 10k -> 10K
- R6: value 10K -> 10k
- R8: value (none) -> 1K
- U1: value LM4040 -> TMPM04215; device PSU200A_Ctrl:TO92- -> myLibs:TMPM04XXX
- moved C1 88.7 mm to (2.54, -64.8)
- moved X4 86.1 mm to (95.0, 62.0), turned to 270 degrees
- moved X2 84.9 mm to (5.00, 25.0)
- moved C2 61.3 mm to (2.54, -58.4)
- moved TP6 54.2 mm to (94.8, 69.5)
- moved C3 52.3 mm to (22.9, 21.6)
- moved R8 47.8 mm to (75.7, 70.1), turned to 180 degrees
- moved TP5 40.6 mm to (61.1, 65.2)
- moved U1 40.5 mm to (11.4, 52.1)
- moved C6 37.1 mm to (68.9, 74.6), turned to 270 degrees
- moved R5 33.9 mm to (40.6, 43.2)
- moved R7 33.9 mm to (48.3, 10.2)
- moved C5 31.4 mm to (61.6, 57.8), turned to 90 degrees
- moved X1 30.8 mm to (5.00, 40.0), flipped to the bottom, turned to 270 degrees
- moved TP7 26.9 mm to (36.0, 45.5)
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Connections:
- removed net N$14: C5.1, R8.1
- removed net N$16: C4.2, C5.2, U1.3
- removed net V+: IC1.8, IC2.8
- removed net V-: IC1.4, IC2.4
- new net +15V: C10.1, C12.1, C2.1, C4.+, C6.1, IC1.8, IC2.8, R8.1, TP3.TP, U1.P$3, X5.3
- new net -15V: C1.1, C11.1, C5.-, C7.2, IC1.4, IC2.4, TP1.TP, U1.P$5, X5.4
- new net N$13: U1.P$7, X3.1
- new net N$15: U1.P$6, X3.2
- new net PE: X3.3
- net +10V: now also C13.1, U2.2, X1.1; no longer C4.1, U1.2
- net GND: now also C1.2, C10.2, C11.2, C12.2, C13.2, C2.2, C4.-, C5.+, C6.2, C7.1, D1.C, TP2.TP, U1.P$4, U2.3, X1.3, X4.3; no longer X2.3
- net N$1: now also X1.2; no longer X3.2
- net N$10: now also R6.2; no longer R4.2
- net N$11: now also C8.2, R4.2, R6.1; no longer C2.2, R4.1, R6.2
- net N$12: now also C8.1, R4.1, X2.2; no longer C2.1, R6.1, X4.2
- net N$17: now also R7.2; no longer R5.2
- net N$18: now also C9.2, R5.2, R7.1; no longer C3.2, R5.1, R7.2
- net N$3: now also C3.1; no longer C1.1
- net N$4: now also C3.2; no longer C1.2
- net N$5: now also X2.1; no longer X4.1
- net N$6: now also C9.1, R5.1, X2.3; no longer C3.1, R7.1, X4.3
- net N$7: now also D1.A, TP7.TP
- net N$8: now also TP6.TP, X4.1; no longer X2.1
- net N$9: now also X4.2; no longer X2.2
Routing:
- net GND: track 0.00 -> 65.0 mm
- net -15V: track 0.00 -> 39.1 mm
- net +15V: track 0.00 -> 30.7 mm
- net N$15: track 0.00 -> 28.6 mm
- net N$13: track 0.00 -> 18.8 mm
- net +10V: track 0.00 -> 6.31 mm
- added copper zone on layer 16, net GND
