File: PSU200A_Ctrl.sch (EAGLE design)
At the start: 30 parts, among them IC1 LM358D, IC2 LM358D, U1 LM4040

Commit message: schematic done
Parts:
- added C10, C11, C12, C13, C7: 0.1u, rcl:C-EUC1206
- added C8, C9: 1n, rcl:C-EUC1206
- added D1: 1N4148DO35-7, diode:1N4148DO35-7
- added U2: LM4040, PSU200A_Ctrl:LM4040
- C1: value 2.2u -> 0.1u
- C2: value 1n -> 0.1u
- C3: value 1n -> 2.2u
- C4, C5: value (none) -> 22u; device rcl:C-EUC1206 -> rcl:CPOL-EUB
- C6: value (none) -> 0.1u
- R4: value 10k -> 10K
- R6: value 10K -> 10k
- R8: value (none) -> 1K
- U1: value LM4040 -> TMPM04215; device PSU200A_Ctrl:LM4040 -> myLibs:TMPM04215
Connections:
- removed net N$14: C5.1, R8.1
- removed net N$16: C4.2, C5.2, U1.A
- new net +15V: C10.1, C12.1, C2.1, C4.+, C6.1, IC1P.V+, IC2P.V+, R8.1, TP3.TP, U1.VOUT_1, X5-3.1
- new net -15V: C1.1, C11.1, C5.-, C7.2, IC1P.V-, IC2P.V-, TP1.TP, U1.VOUT_2, X5-4.1
- new net N$13: U1.AC_L, X3-1.1
- new net N$15: U1.AC_N, X3-2.1
- new net PE: X3-3.1
- net +10V: now also C13.1, U2.C, X1-1.1; no longer C4.1, U1.C
- net GND: now also C1.2, C10.2, C11.2, C12.2, C13.2, C2.2, C4.-, C5.+, C6.2, C7.1, D1.C, TP2.TP, U1.COM, U2.A, X1-3.1, X4-3.1; no longer X2-3.1
- net N$1: now also X1-2.1; no longer X3-2.1
- net N$10: now also R6.2; no longer R4.2
- net N$11: now also C8.2, R4.2, R6.1; no longer C2.2, R4.1, R6.2
- net N$12: now also C8.1, R4.1, X2-2.1; no longer C2.1, R6.1, X4-2.1
- net N$17: now also R7.2; no longer R5.2
- net N$18: now also C9.2, R5.2, R7.1; no longer C3.2, R5.1, R7.2
- net N$3: now also C3.1; no longer C1.1
- net N$4: now also C3.2; no longer C1.2
- net N$5: now also X2-1.1; no longer X4-1.1
- net N$6: now also C9.1, R5.1, X2-3.1; no longer C3.1, R7.1, X4-3.1
- net N$7: now also D1.A, TP7.TP
- net N$8: now also TP6.TP, X4-1.1; no longer X2-1.1
- net N$9: now also X4-2.1; no longer X2-2.1
Other:
- moved on the sheet: C1, C2, C3, C6, IC1A, IC1B, IC2A, IC2B, OK1, R1, R2, R3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
